Commit message: control

File: hercules/hercules_description/urdf/hercules.urdf.xacro (robot description, xacro)
@@ -9,4 +9,5 @@
   <xacro:property name="track" value="0.17" />
   <xacro:property name="wheel_vertical_offset" value="0.0" />
+  <xacro:property name="PI" value="3.14159265359" />
  <material name="black"><color rgba="0.15 0.15 0.15 1" /></material>
   <link name="base_link">
@@ -19,11 +20,17 @@
       </material>
     </visual>
+    <collision>
+      <origin xyz="0 0 0" rpy="$0 0 0"/>
+      <geometry>
+        <box size="${chassis_length} ${chassis_width} ${chassis_height}"/>
+      </geometry>
+    </collision>
     <inertial>
         <origin xyz="0 0 0" rpy="0 0 0"/>
-        <mass value="1.5"/>
+        <mass value="1.8"/>
         <inertia
-          ixx="0.0024" ixy="0" ixz="0"
-          iyy="0.0054" iyz="0"
-          izz="0.0075"/>
+          ixx="0.0029" ixy="0" ixz="0"
+          iyy="0.0065" iyz="0"
+          izz="0.0091"/>
     </inertial>
   </link>
@@ -31,130 +38,61 @@
       <material>Gazebo/Green</material>
   </gazebo>
-  <link name="front_right_wheel">
-    <visual>
-      <geometry>
-        <!-- Example of where mesh definition goes (replaces cylinder) -->
-        <!-- <mesh filename="package://hercules_description/meshes/Wheels.dae"/> -->
-        <cylinder radius="${wheel_radius}" length="${wheel_width}"/>
-      </geometry>
-      <material name="black" />
-    </visual>
-    <collision>
-      <geometry>
-        <cylinder radius="${wheel_radius}" length="${wheel_width}"/>
-      </geometry>
-      <material name="black" />
-    </collision>
-    <inertial>
+  <xacro:macro name="wheel" params="prefix *joint_pose">
+    <link name="${prefix}_wheel">
+      <visual>
+        <origin xyz="0 0 0" rpy="${PI/2} 0 0"/>
+        <geometry>
+          <cylinder radius="${wheel_radius}" length="${wheel_width}"/>
+        </geometry>
+        <material name="black" />
+      </visual>
+      <collision>
+        <origin xyz="0 0 0" rpy="${PI/2} 0 0"/>
+        <geometry>
+          <cylinder radius="${wheel_radius}" length="${wheel_width}"/>
+        </geometry>
+      </collision>
+      <inertial>
         <origin xyz="0 0 0" rpy="0 0 0"/>
         <mass value="0.05"/>
         <inertia
           ixx="2.6326e-5" ixy="0" ixz="0"
-          iyy="2.6326e-5" iyz="0"
-          izz="4.5156e-5"/>
-    </inertial>
-  </link>
-  <gazebo reference="front_right_wheel">
+          iyy="4.5156e-5" iyz="0"
+          izz="2.6326e-5"/>
+      </inertial>
+    </link>
+    <gazebo reference="${prefix}_wheel">
       <material>Gazebo/DarkGrey</material>
-  </gazebo>
-  <joint name="front_right_wheel_joint" type="continuous">
-    <axis xyz="0 0 1"/>
-    <parent link="base_link"/>
-    <child link="front_right_wheel"/>
-    <origin rpy="-1.5708 0 0" xyz="${wheelbase/2} ${-track/2} ${wheel_vertical_offset}"/>
-  </joint>
-  <link name="front_left_wheel">
-    <visual>
-      <geometry>
-        <cylinder radius="${wheel_radius}" length="${wheel_width}"/>
-      </geometry>
-      <material name="black" />
-    </visual>
-    <collision>
-      <geometry>
-        <cylinder radius="${wheel_radius}" length="${wheel_width}"/>
-      </geometry>
-      <material name="black" />
-    </collision>
-    <inertial>
-        <origin xyz="0 0 0" rpy="0 0 0"/>
-        <mass value="0.05"/>
-        <inertia
-          ixx="2.6326e-5" ixy="0" ixz="0"
-          iyy="2.6326e-5" iyz="0"
-          izz="4.5156e-5"/>
-    </inertial>
-  </link>
-  <gazebo reference="front_left_wheel">
-      <material>Gazebo/DarkGrey</material>
-  </gazebo>
-  <joint name="front_left_wheel_joint" type="continuous">
-    <axis xyz="0 0 1"/>
-    <parent link="base_link"/>
-    <child link="front_left_wheel"/>
-    <origin rpy="-1.5708 0 0" xyz="${wheelbase/2} ${track/2} ${wheel_vertical_offset}"/>
-  </joint>
-  <link name="back_right_wheel">
-    <visual>
-      <geometry>
-        <cylinder radius="${wheel_radius}" length="${wheel_width}"/>
-      </geometry>
-      <material name="black" />
-    </visual>
-    <collision>
-      <geometry>
-        <cylinder radius="${wheel_radius}" length="${wheel_width}"/>
-      </geometry>
-      <material name="black" />
-    </collision>
-    <inertial>
-        <origin xyz="0 0 0" rpy="0 0 0"/>
-        <mass value="0.05"/>
-        <inertia
-          ixx="2.6326e-5" ixy="0" ixz="0"
-          iyy="2.6326e-5" iyz="0"
-          izz="4.5156e-5"/>
-    </inertial>
-  </link>
-  <gazebo reference="back_right_wheel">
-      <material>Gazebo/DarkGrey</material>
-  </gazebo>
-  <joint name="back_right_wheel_joint" type="continuous">
-    <axis xyz="0 0 1"/>
-    <parent link="base_link"/>
-    <child link="back_right_wheel"/>
-    <origin rpy="-1.5708 0 0" xyz="${-wheelbase/2} ${-track/2} ${wheel_vertical_offset}"/>
-  </joint>
-  <link name="back_left_wheel">
-    <visual>
-      <geometry>
-        <cylinder radius="${wheel_radius}" length="${wheel_width}"/>
-      </geometry>
-      <material name="black" />
-    </visual>
-    <collision>
-      <geometry>
-        <cylinder radius="${wheel_radius}" length="${wheel_width}"/>
-      </geometry>
-      <material name="black" />
-    </collision>
-    <inertial>
-        <origin xyz="0 0 0" rpy="0 0 0"/>
-        <mass value="0.05"/>
-        <inertia
-          ixx="2.6326e-5" ixy="0" ixz="0"
-          iyy="2.6326e-5" iyz="0"
-          izz="4.5156e-5"/>
-    </inertial>
-  </link>
-  <gazebo reference="back_left_wheel">
-      <material>Gazebo/DarkGrey</material>
-  </gazebo>
-  <joint name="back_left_wheel_joint" type="continuous">
-    <axis xyz="0 0 1"/>
-    <parent link="base_link"/>
-    <child link="back_left_wheel"/>
-    <origin rpy="-1.5708 0 0" xyz="${-wheelbase/2} ${track/2} ${wheel_vertical_offset}"/>
-  </joint>
+    </gazebo>
+    <joint name="${prefix}_wheel_joint" type="continuous">
+      <parent link="base_link"/>
+      <child link="${prefix}_wheel" />
+      <xacro:insert_block name="joint_pose" />
+      <axis xyz="0 1 0" />
+    </joint>
+    <!-- In reality, Jackal has only two motors, one per side. However, it's more
+         straightforward for Gazebo to simulate as if there's an actuator per wheel. -->
+    <transmission name="${prefix}_wheel_trans">
+      <type>transmission_interface/SimpleTransmission</type>
+      <joint name="${prefix}_wheel_joint">
+        <hardwareInterface>VelocityJointInterface</hardwareInterface>
+      </joint>
+      <actuator name="${prefix}_actuator">
+        <mechanicalReduction>1</mechanicalReduction>
+      </actuator>
+    </transmission>
+  </xacro:macro>
+  <xacro:wheel prefix="front_left">
+    <origin xyz="${wheelbase/2} ${track/2} ${wheel_vertical_offset}" rpy="0 0 0" />
+  </xacro:wheel>
+  <xacro:wheel prefix="front_right">
+    <origin xyz="${wheelbase/2} ${-track/2} ${wheel_vertical_offset}" rpy="0 0 0" />
+  </xacro:wheel>
+  <xacro:wheel prefix="back_left">
+    <origin xyz="${-wheelbase/2} ${track/2} ${wheel_vertical_offset}" rpy="0 0 0" />
+  </xacro:wheel>
+  <xacro:wheel prefix="back_right">
+    <origin xyz="${-wheelbase/2} ${-track/2} ${wheel_vertical_offset}" rpy="0 0 0" />
+  </xacro:wheel>
   <!-- Bring in simulation data for Gazebo. -->
   <xacro:include filename="$(find hercules_description)/urdf/hercules.gazebo" />

Commit message: raspberry pi

File: hercules/hercules_description/urdf/hercules.urdf.xacro (robot description, xacro)
@@ -21,5 +21,5 @@
     </visual>
     <collision>
-      <origin xyz="0 0 0" rpy="$0 0 0"/>
+      <origin xyz="0 0 0" rpy="0 0 0"/>
       <geometry>
         <box size="${chassis_length} ${chassis_width} ${chassis_height}"/>
@@ -35,8 +35,63 @@
     </inertial>
   </link>
-  <gazebo reference="base_link">
-      <material>Gazebo/Green</material>
-  </gazebo>
-  <xacro:macro name="wheel" params="prefix *joint_pose">
+  <link name="top_mount">
+    <visual>
+      <geometry>
+        <box size="${chassis_length} ${chassis_width} 0.002"/>
+      </geometry>
+      <material name="green">
+        <color rgba="0.22 1.0 0.07 1"/>
+      </material>
+    </visual>
+  </link>
+  <joint name="top_mount_joint" type="fixed">
+    <axis xyz="0 1 0" />
+    <origin xyz="0 0 ${chassis_height/2 + 0.04}" rpy="0 0 0"/>
+    <parent link="base_link"/>
+    <child link="top_mount"/>
+  </joint>
+  <link name="battery">
+    <visual>
+      <geometry>
+        <box size="0.19 0.08 0.02"/>
+      </geometry>
+      <material name="silver">
+        <color rgba="0.75 0.75 0.75 1"/>
+      </material>
+    </visual>
+  </link>
+  <joint name="battery_joint" type="fixed">
+    <axis xyz="0 1 0" />
+    <origin xyz="0.015 0 0.01" rpy="0 0 0"/>
+    <parent link="top_mount"/>
+    <child link="battery"/>
+  </joint>
+   <link name="laser">
+    <collision>
+      <origin xyz="0 0 0" rpy="0 0 0"/>
+      <geometry>
+        <box size="0.05 0.05 0.05"/>
+      </geometry>
+    </collision>
+    <visual>
+      <origin xyz="0 0 0" rpy="0 0 0"/>
+      <geometry>
+        <box size="0.05 0.05 0.05"/>
+      </geometry>
+      <material name="black"><color rgba="0.15 0.15 0.15 1" /></material>
+    </visual>
+    <inertial>
+      <mass value="1e-5" />
+      <origin xyz="0 0 0" rpy="0 0 0"/>
+      <inertia ixx="1e-6" ixy="0" ixz="0" iyy="1e-6" iyz="0" izz="1e-6" />
+    </inertial>
+  </link>
+  <joint name="laser_joint" type="fixed">
+    <axis xyz="0 1 0" />
+    <origin xyz="0 0 0.025" rpy="0 0 0"/>
+    <parent link="battery"/>
+    <child link="laser"/>
+  </joint>
+<xacro:macro name="wheel" params="prefix *joint_pose">
     <link name="${prefix}_wheel">
       <visual>
@@ -71,6 +126,4 @@
       <axis xyz="0 1 0" />
     </joint>
-    <!-- In reality, Jackal has only two motors, one per side. However, it's more
-         straightforward for Gazebo to simulate as if there's an actuator per wheel. -->
     <transmission name="${prefix}_wheel_trans">
       <type>transmission_interface/SimpleTransmission</type>
@@ -95,5 +148,36 @@
     <origin xyz="${-wheelbase/2} ${-track/2} ${wheel_vertical_offset}" rpy="0 0 0" />
   </xacro:wheel>
+  <xacro:macro name="offset" params="prefix *offset_pose">
+    <link name="${prefix}_offset">
+      <visual>
+        <origin xyz="0 0 0" rpy="0 0 0"/>
+        <geometry>
+          <cylinder radius="0.0025" length="0.043"/>
+        </geometry>
+        <material name="gold">
+           <color rgba="0.83 0.68 0.0 1"/>
+        </material>
+      </visual>
+    </link>
+    <joint name="${prefix}_offset_joint" type="fixed">
+      <parent link="base_link"/>
+      <child link="${prefix}_offset" />
+      <xacro:insert_block name="offset_pose" />
+      <axis xyz="0 1 0" />
+    </joint>
+  </xacro:macro>
+  <xacro:offset prefix="front_left">
+    <origin xyz="${0.175/2} ${0.12/2} 0.035" rpy="0 0 0" />
+  </xacro:offset>
+  <xacro:offset prefix="front_right">
+    <origin xyz="${0.175/2} ${-0.12/2} 0.035" rpy="0 0 0" />
+  </xacro:offset>
+  <xacro:offset prefix="back_left">
+    <origin xyz="${-0.175/2} ${0.12/2} 0.035" rpy="0 0 0" />
+  </xacro:offset>
+  <xacro:offset prefix="back_right">
+    <origin xyz="${-0.175/2} ${-0.12/2} 0.035" rpy="0 0 0" />
+  </xacro:offset>
   <!-- Bring in simulation data for Gazebo. -->
-  <xacro:include filename="$(find hercules_description)/urdf/hercules.gazebo" />
+  <!-- <xacro:include filename="$(find hercules_description)/urdf/hercules.gazebo" /> -->
 </robot>

Commit message: got closed loop control using ros_control working. readme

File: hercules/hercules_description/urdf/hercules.urdf.xacro (robot description, xacro)
@@ -20,18 +20,4 @@
       </material>
     </visual>
-    <collision>
-      <origin xyz="0 0 0" rpy="0 0 0"/>
-      <geometry>
-        <box size="${chassis_length} ${chassis_width} ${chassis_height}"/>
-      </geometry>
-    </collision>
-    <inertial>
-        <origin xyz="0 0 0" rpy="0 0 0"/>
-        <mass value="1.8"/>
-        <inertia
-          ixx="0.0029" ixy="0" ixz="0"
-          iyy="0.0065" iyz="0"
-          izz="0.0091"/>
-    </inertial>
   </link>
   <link name="top_mount">
@@ -94,5 +80,5 @@
   </joint>
 <xacro:macro name="wheel" params="prefix *joint_pose">
-    <link name="${prefix}_wheel">
+    <link name="${prefix}_wheel_link">
       <visual>
         <origin xyz="0 0 0" rpy="${PI/2} 0 0"/>
@@ -117,10 +103,10 @@
       </inertial>
     </link>
-    <gazebo reference="${prefix}_wheel">
+    <gazebo reference="${prefix}_wheel_link">
       <material>Gazebo/DarkGrey</material>
     </gazebo>
-    <joint name="${prefix}_wheel_joint" type="continuous">
+    <joint name="${prefix}_wheel" type="continuous">
       <parent link="base_link"/>
-      <child link="${prefix}_wheel" />
+      <child link="${prefix}_wheel_link" />
       <xacro:insert_block name="joint_pose" />
       <axis xyz="0 1 0" />
@@ -128,6 +114,6 @@
     <transmission name="${prefix}_wheel_trans">
       <type>transmission_interface/SimpleTransmission</type>
-      <joint name="${prefix}_wheel_joint">
-        <hardwareInterface>VelocityJointInterface</hardwareInterface>
+      <joint name="${prefix}_wheel">
+        <hardwareInterface>hardware_interface/VelocityJointInterface</hardwareInterface>
       </joint>
       <actuator name="${prefix}_actuator">

Commit message: fixed simulation

File: hercules/hercules_description/urdf/hercules.urdf.xacro (robot description, xacro)
@@ -11,5 +11,11 @@
   <xacro:property name="PI" value="3.14159265359" />
  <material name="black"><color rgba="0.15 0.15 0.15 1" /></material>
-  <link name="base_link">
+  <link name="base_link"></link>
+  <joint name="base_link_joint" type="fixed">
+    <origin xyz="0 0 0" rpy="0 0 0" />
+    <parent link="base_link"/>
+    <child link="chassis_link" />
+  </joint>
+   <link name="chassis_link">
     <visual>
       <geometry>
@@ -20,4 +26,20 @@
       </material>
     </visual>
+     <collision>
+      <origin xyz="0 0 ${chassis_height/2}"/>
+      <geometry>
+        <box size="${chassis_length} ${chassis_width} ${chassis_height}"/>
+      </geometry>
+    </collision>
+    <inertial>
+      <!-- Center of mass -->
+      <origin xyz="0.012  0.002 0.067" rpy="0 0 0"/>
+      <mass value="1.5"/>
+      <!-- Moments of inertia: ( chassis without wheels ) -->
+      <inertia
+        ixx="0.3136" ixy="-0.0008" ixz="0.0164"
+        iyy="0.3922" iyz="-0.0009"
+        izz="0.4485"/>
+</inertial>
   </link>
   <link name="top_mount">
@@ -34,5 +56,5 @@
     <axis xyz="0 1 0" />
     <origin xyz="0 0 ${chassis_height/2 + 0.04}" rpy="0 0 0"/>
-    <parent link="base_link"/>
+    <parent link="chassis_link"/>
     <child link="top_mount"/>
   </joint>
@@ -107,5 +129,5 @@
     </gazebo>
     <joint name="${prefix}_wheel" type="continuous">
-      <parent link="base_link"/>
+      <parent link="chassis_link"/>
       <child link="${prefix}_wheel_link" />
       <xacro:insert_block name="joint_pose" />
@@ -147,5 +169,5 @@
     </link>
     <joint name="${prefix}_offset_joint" type="fixed">
-      <parent link="base_link"/>
+      <parent link="chassis_link"/>
       <child link="${prefix}_offset" />
       <xacro:insert_block name="offset_pose" />
@@ -166,4 +188,4 @@
   </xacro:offset>
   <!-- Bring in simulation data for Gazebo. -->
-  <!-- <xacro:include filename="$(find hercules_description)/urdf/hercules.gazebo" /> -->
+  <xacro:include filename="$(find hercules_description)/urdf/hercules.gazebo" />
 </robot>
